File: ATMEGA328-Motor-Board/pcb/ATMEGA328_Motor_Board.kicad_pcb (KiCad board)
At the start: 2 copper layers, 77 x 100 mm, 259 parts, among them P1 CONN_01X04, P10 CONN_01X04, P11 CONN_01X02, P12 CONN_01X03, P13 CONN_01X02, P14 USB_MINI, P15 CONN_01X03, P16 CONN_02X03, P2 CONN_01X04, P3 CONN_01X03, P4 CONN_01X03, P5 CONN_01X03, P6 CONN_01X03, P7 CONN_01X03, P8 CONN_01X03, P9 CONN_01X04, SW1 Pulsador_2p, U1 ATMEGA328, U10 VOM617A, U11 VOM617A, U12 ASSR-1218, U13 ASSR-1218, U2 PCA9685, U3 FT231X, U4 L298P, U5 L298P, U6 TSR_1, U7 LM2903, U8 LM2903, U9 VOM617A, Y1 16MHz

Commit message: two
Parts:
- removed JP2: JUMPER_3, Conectores:Pin_Header_Straight_1x03
Changed lines of the file:
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@@
-(kicad_pcb (version 4) (host pcbnew 4.1.0-alpha+201608101232+7015~46~ubuntu14.04.1-product)
+(kicad_pcb (version 20171130) (host pcbnew "(5.1.5-0-10_14)")
   (general
-    (links 498)
-    (no_connects 0)
-    (area 107.477343 35.3127 186.633134 142.4973)
     (thickness 1.6)
     (drawings 98)
     (tracks 4270)
     (zones 0)
-    (modules 259)
+    (modules 258)
     (nets 126)
   )
@@
     (zone_45_only no)
     (trace_min 0.2)
-    (segment_width 0.2)
-    (edge_width 0.15)
     (via_size 0.8)
     (via_drill 0.4)
@@
     (uvia_min_size 0)
     (uvia_min_drill 0)
+    (edge_width 0.15)
+    (segment_width 0.2)
     (pcb_text_width 0.3)
     (pcb_text_size 1.5 1.5)
@@
       (layerselection 0x00000_7fffffff)
       (usegerberextensions true)
+      (usegerberattributes false)
+      (usegerberadvancedattributes false)
+      (creategerberjobfile false)
       (excludeedgelayer true)
       (linewidth 0.100000)
@@
       (hpglpennumber 1)
       (hpglpenspeed 20)
-      (hpglpendiameter 15)
+      (hpglpendiameter 15.000000)
       (psnegative false)
       (psa4output false)
@@
       (drillshape 0)
       (scaleselection 1)
-      (outputdirectory gerber/))
+      (outputdirectory "gerber/"))
   )
   (net 0 "")
@@
     (at 178.54 120.55 270)
     (fp_text reference G*** (at 0 0 270) (layer B.SilkS) hide
-      (effects (font (thickness 0.3)) (justify mirror))
+      (effects (font (size 1.524 1.524) (thickness 0.3)) (justify mirror))
     )
     (fp_text value LOGO (at 0.75 0 270) (layer B.SilkS) hide
-      (effects (font (thickness 0.3)) (justify mirror))
+      (effects (font (size 1.524 1.524) (thickness 0.3)) (justify mirror))
     )
     (fp_poly (pts (xy -3.247962 -2.471678) (xy -3.173547 -2.504764) (xy -3.109752 -2.553719) (xy -3.060672 -2.617347)
@@
     (at 118.89 57.11 270)
     (fp_text reference G*** (at 0 0 270) (layer B.SilkS) hide
-      (effects (font (thickness 0.3)) (justify mirror))
+      (effects (font (size 1.524 1.524) (thickness 0.3)) (justify mirror))
     )
     (fp_text value LOGO (at 0.75 0 270) (layer B.SilkS) hide
-      (effects (font (thickness 0.3)) (justify mirror))
+      (effects (font (size 1.524 1.524) (thickness 0.3)) (justify mirror))
     )
     (fp_poly (pts (xy 0.169564 -3.124473) (xy 0.426341 -3.147656) (xy 0.580722 -3.188216) (xy 0.619355 -3.222625)
@@
       (net 1 GND))
     (model Pin_Headers.3dshapes/Pin_Header_Straight_1x03.wrl
-      (at (xyz 0 -0.1 0))
+      (offset (xyz 0 -2.539999961853027 0))
       (scale (xyz 1 1 1))
       (rotate (xyz 0 0 90))
@@
       (net 1 GND))
     (model Pin_Headers.3dshapes/Pin_Header_Straight_1x03.wrl
-      (at (xyz 0 -0.1 0))
+      (offset (xyz 0 -2.539999961853027 0))
       (scale (xyz 1 1 1))
       (rotate (xyz 0 0 90))
@@
       (net 1 GND))
     (model Pin_Headers.3dshapes/Pin_Header_Straight_1x03.wrl
-      (at (xyz 0 -0.1 0))
+      (offset (xyz 0 -2.539999961853027 0))
       (scale (xyz 1 1 1))
       (rotate (xyz 0 0 90))
@@
       (net 1 GND))
     (model Pin_Headers.3dshapes/Pin_Header_Straight_1x03.wrl
-      (at (xyz 0 -0.1 0))
+      (offset (xyz 0 -2.539999961853027 0))
       (scale (xyz 1 1 1))
       (rotate (xyz 0 0 90))
@@
       (net 52 +24V))
     (model Pin_Headers.3dshapes/Pin_Header_Straight_1x03.wrl
-      (at (xyz 0 -0.1 0))
+      (offset (xyz 0 -2.539999961853027 0))
       (scale (xyz 1 1 1))
       (rotate (xyz 0 0 90))
@@
       (net 52 +24V))
     (model Pin_Headers.3dshapes/Pin_Header_Straight_1x03.wrl
-      (at (xyz 0 -0.1 0))
+      (offset (xyz 0 -2.539999961853027 0))
       (scale (xyz 1 1 1))
       (rotate (xyz 0 0 90))
@@
       (net 50 "Net-(JP4-Pad3)"))
     (model Pin_Headers.3dshapes/Pin_Header_Straight_1x03.wrl
-      (at (xyz 0 -0.1 0))
+      (offset (xyz 0 -2.539999961853027 0))
       (scale (xyz 1 1 1))
       (rotate (xyz 0 0 90))
@@
       (net 49 "Net-(JP3-Pad3)"))
     (model Pin_Headers.3dshapes/Pin_Header_Straight_1x03.wrl
-      (at (xyz 0 -0.1 0))
-      (scale (xyz 1 1 1))
-      (rotate (xyz 0 0 90))
-    )
-  )
-  (module Conectores:Pin_Header_Straight_1x03 (layer F.Cu)
-    (at 146.83 54.02)
-    (descr "Through hole pin header")
-    (tags "pin header")
-    (fp_text reference JP2 (at 0 7.3) (layer F.SilkS)
-      (effects (font (size 0.8 0.8) (thickness 0.15)))
-    )
-    (fp_text value JUMPER_3 (at 0 -3.1) (layer F.Fab)
-      (effects (font (size 1 1) (thickness 0.15)))
-    )
-    (fp_line (start -1.75 -1.75) (end -1.75 6.85) (layer F.CrtYd) (width 0.05))
-    (fp_line (start 1.75 -1.75) (end 1.75 6.85) (layer F.CrtYd) (width 0.05))
-    (fp_line (start -1.75 -1.75) (end 1.75 -1.75) (layer F.CrtYd) (width 0.05))
-    (fp_line (start -1.75 6.85) (end 1.75 6.85) (layer F.CrtYd) (width 0.05))
-    (fp_line (start -1.27 1.27) (end -1.27 6.35) (layer F.SilkS) (width 0.15))
-    (fp_line (start -1.27 6.35) (end 1.27 6.35) (layer F.SilkS) (width 0.15))
-    (fp_line (start 1.27 6.35) (end 1.27 1.27) (layer F.SilkS) (width 0.15))
-    (fp_line (start 1.55 -1.55) (end 1.55 0) (layer F.SilkS) (width 0.15))
-    (fp_line (start 1.27 1.27) (end -1.27 1.27) (layer F.SilkS) (width 0.15))
-    (fp_line (start -1.55 0) (end -1.55 -1.55) (layer F.SilkS) (width 0.15))
-    (fp_line (start -1.55 -1.55) (end 1.55 -1.55) (layer F.SilkS) (width 0.15))
-    (pad 1 thru_hole rect (at 0 0) (size 2.032 1.7272) (drill 1) (layers *.Cu *.Mask F.SilkS)
-      (net 43 ENC1_B2))
-    (pad 2 thru_hole oval (at 0 2.54) (size 2.032 1.7272) (drill 1) (layers *.Cu *.Mask F.SilkS)
-      (net 28 ENC1_B))
-    (pad 3 thru_hole oval (at 0 5.08) (size 2.032 1.7272) (drill 1) (layers *.Cu *.Mask F.SilkS)
-      (net 48 "Net-(JP2-Pad3)"))
-    (model Pin_Headers.3dshapes/Pin_Header_Straight_1x03.wrl
-      (at (xyz 0 -0.1 0))
+      (offset (xyz 0 -2.539999961853027 0))
       (scale (xyz 1 1 1))
       (rotate (xyz 0 0 90))
@@
       (net 47 "Net-(JP1-Pad3)"))
     (model Pin_Headers.3dshapes/Pin_Header_Straight_1x03.wrl
-      (at (xyz 0 -0.1 0))
+      (offset (xyz 0 -2.539999961853027 0))
       (scale (xyz 1 1 1))
       (rotate (xyz 0 0 90))
@@
       (net 1 GND))
     (model Pin_Headers.3dshapes/Pin_Header_Straight_2x03.wrl
-      (at (xyz 0.05 -0.1 0))
+      (offset (xyz 1.269999980926514 -2.539999961853027 0))
       (scale (xyz 1 1 1))
       (rotate (xyz 0 0 90))
@@
       (net 52 +24V))
     (model Pin_Headers.3dshapes/Pin_Header_Straight_1x02.wrl
-      (at (xyz 0 -0.05 0))
+      (offset (xyz 0 -1.269999980926514 0))
       (scale (xyz 1 1 1))
       (rotate (xyz 0 0 90))
@@
     )
     (polygon
-      (pts        (xy 119.981835 137.789793) (xy 120.32 137.788817) (xy 120.32 132.96) (xy 120.821182 132.959663) (xy 120.64 92.23)
+      (pts
+        (xy 119.981835 137.789793) (xy 120.32 137.788817) (xy 120.32 132.96) (xy 120.821182 132.959663) (xy 120.64 92.23)
         (xy 147.88 92.23) (xy 147.77 97.2) (xy 147.34 137.21) (xy 135.244746 137.200872) (xy 135.25 137.7)
         (xy 148.07 137.71) (xy 148.18 92.13) (xy 174.605 92.3) (xy 174.78 123.69) (xy 177.68 126.39)
@@
     )
     (polygon
-      (pts        (xy 120.13 90.85) (xy 120.205 131.525) (xy 120.52 131.67) (xy 120.37 92.25) (xy 147.919632 92.218168)
+      (pts
+        (xy 120.13 90.85) (xy 120.205 131.525) (xy 120.52 131.67) (xy 120.37 92.25) (xy 147.919632 92.218168)
         (xy 147.931322 137.088168) (xy 137.270796 137.088168) (xy 137.281322 137.688168) (xy 148.38 137.77) (xy 148.378678 92.211832)
         (xy 174.53 92.28) (xy 174.781322 123.688168) (xy 177.681322 126.388168) (xy 177.631322 138.738168) (xy 137.181322 138.950133)
